Commit message: Add origin and collide_bitmask

File: urdf/geometry.xacro (robot description, xacro)
@@ -5,8 +5,8 @@
   <!-- Box -->
   <!-- This macro should not be named box, because this leads to naming collisions with the build in box element -->
-  <xacro:macro name="gbox" params="name mass sx sy sz cmask:=0x00 xyz:='0 0 0' rpy='0 0 0'">
+  <xacro:macro name="gbox" params="name mass sx sy sz *origin *collide_bitmask">
     <link name="${name}">
       <visual>
-        <origin xyz="${xyz}" rpy="${rpy}" />
+        <xacro:insert_block name="origin" />
         <geometry>
           <box size="${sx} ${sy} ${sz}" />
@@ -14,5 +14,5 @@
       </visual>
       <collision>
-        <origin xyz="${xyz}" rpy="${rpy}" />
+        <xacro:insert_block name="origin" />
         <geometry>
           <box size="${sx} ${sy} ${sz}" />
@@ -28,6 +28,5 @@
         <surface>
           <contact>
-            <!-- <collide_bitmask>"${cmask}"</collide_bitmask> -->
-            <!-- <xacro:insert_block name="${cmask}" /> -->
+            <xacro:insert_block name="collide_bitmask" />
           </contact>
         </surface>
@@ -37,8 +36,8 @@
   <!-- Cylinder -->
   <!-- This macro should not be named cylinder, because this leads to naming collisions with the build in cylinder element -->
-  <xacro:macro name="gcylinder" params="name mass length radius cmask:=0x00 xyz='0 0 0' rpy='0 0 0'">
+  <xacro:macro name="gcylinder" params="name mass length radius *origin *collide_bitmask">
     <link name="${name}">
       <visual>
-        <origin xyz="${xyz}" rpy="${rpy}" />
+        <xacro:insert_block name="origin" />
         <geometry>
           <cylinder length="${length}" radius="${radius}" />
@@ -46,5 +45,5 @@
       </visual>
       <collision>
-        <origin xyz="${xyz}" rpy="${rpy}" />
+        <xacro:insert_block name="origin" />
         <geometry>
           <cylinder length="${length}" radius="${radius}" />
@@ -60,6 +59,5 @@
         <surface>
           <contact>
-            <!-- <collide_bitmask>"${cmask}"</collide_bitmask> -->
-            <!-- <xacro:insert_block name="${cmask}" /> -->
+            <xacro:insert_block name="collide_bitmask" />
           </contact>
         </surface>
@@ -70,8 +68,8 @@
   <!-- This macro should not be named sphere, because this leads to naming collisions
        with the build in sphere element -->
-  <xacro:macro name="gsphere" params="name mass radius cmask:=0x00 xyz='0 0 0' rpy='0 0 0'">
+  <xacro:macro name="gsphere" params="name mass radius *origin *collide_bitmask">
     <link name="${name}">
       <visual>
-        <origin xyz="${xyz}" rpy="${rpy}" />
+        <xacro:insert_block name="origin" />
         <geometry>
           <sphere radius="${radius}" />
@@ -79,5 +77,5 @@
       </visual>
       <collision>
-        <origin xyz="${xyz}" rpy="${rpy}" />
+        <xacro:insert_block name="origin" />
         <geometry>
           <sphere radius="${radius}" />
@@ -93,6 +91,5 @@
         <surface>
           <contact>
-            <!-- <collide_bitmask>"${cmask}"</collide_bitmask> -->
-            <!-- <xacro:insert_block name="${cmask}" /> -->
+            <xacro:insert_block name="collide_bitmask" />
           </contact>
         </surface>
